Commit message: second commit

File: CrazyS/rotors_description/urdf/f550.xacro (robot description, xacro)
@@ -21,5 +21,5 @@
   <xacro:property name="rotor_velocity_slowdown_sim" value="10" />
   <xacro:property name="use_mesh_file" value="true" />
-  <xacro:property name="mesh_file" value="package://rotors_description/meshes/f550.dae" />
+  <xacro:property name="mesh_file" value="package://rotors_description/meshes/f550.stl" />
   <xacro:property name="mass" value="1.5" /> <!-- [kg] -->
   <xacro:property name="body_width" value="0.25" /> <!-- [m] -->
